File: matrix.kicad_sch (KiCad schematic)
At the start: 168 parts, among them SW1 SW_Push, SW10 SW_Push, SW11 SW_Push, SW12 SW_Push, SW13 SW_Push, SW14 SW_Push, SW15 SW_Push, SW16 SW_Push, SW17 SW_Push, SW18 SW_Push, SW19 SW_Push, SW2 SW_Push, SW20 SW_Push, SW21 SW_Push, SW22 SW_Push, SW23 SW_Push, SW24 SW_Push, SW25 SW_Push, SW26 SW_Push, SW27 SW_Push, SW28 SW_Push, SW29 SW_Push, SW3 SW_Push, SW30 SW_Push, SW31 SW_Push, SW32 SW_Push, SW33 SW_Push, SW34 SW_Push, SW35 SW_Push, SW36 SW_Push, SW37 SW_Push, SW38 SW_Push, SW39 SW_Push, SW4 SW_Push, SW40 SW_Push, SW41 SW_Push, SW42 SW_Push, SW43 SW_Push, SW44 SW_Push, SW45 SW_Push, SW46 SW_Push, SW47 SW_Push, SW48 SW_Push, SW49 SW_Push, SW5 SW_Push, SW50 SW_Push, SW51 SW_Push, SW52 SW_Push, SW53 SW_Push, SW54 SW_Push, SW55 SW_Push, SW56 SW_Push, SW57 SW_Push, SW58 SW_Push, SW59 SW_Push, SW6 SW_Push, SW60 SW_Push, SW61 SW_Push, SW62 SW_Push, SW63 SW_Push, SW64 SW_Push, SW65 SW_Push, SW66 SW_Push, SW67 SW_Push, SW68 SW_Push, SW69 SW_Push, SW7 SW_Push, SW70 SW_Push, SW71 SW_Push, SW72 SW_Push, SW73 SW_Push, SW74 SW_Push, SW75 SW_Push, SW76 SW_Push, SW77 SW_Push, SW78 SW_Push, SW79 SW_Push, SW8 SW_Push, SW80 SW_Push, SW81 SW_Push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

Commit message: completed pcb
Parts:
- D1, D10, D11, D12, D13, D14, D15, D16, D17, D18, D19, D2, D20, D21, D22, D23, D24, D25, D26, D27, D28, D29, D3, D30, D31, D32, D33, D34, D35, D36, D37, D38, D39, D4, D40, D41, D42, D43, D44, D45, D46, D47, D48, D49, D5, D50, D51, D52, D53, D54, D55, D56, D57, D58, D59, D6, D60, D61, D62, D63, D64, D65, D66, D67, D68, D69, D7, D70, D71, D72, D73, D74, D75, D76, D77, D78, D79, D8, D80, D81, D82, D83, D84, D9: footprint (none) -> Diode_SMD:D_SOD-123
- SW1: value SW_Push -> esc; footprint (none) -> MX_Only:MXOnly-1U
- SW10: value SW_Push -> f9; footprint (none) -> MX_Only:MXOnly-1U
- SW11: value SW_Push -> f10; footprint (none) -> MX_Only:MXOnly-1U
- SW12: value SW_Push -> f11; footprint (none) -> MX_Only:MXOnly-1U
- SW13: value SW_Push -> f12; footprint (none) -> MX_Only:MXOnly-1U
- SW14: value SW_Push -> prtsc/nmlk; footprint (none) -> MX_Only:MXOnly-1U
- SW15: value SW_Push -> pause/scrlk; footprint (none) -> MX_Only:MXOnly-1U
- SW16: value SW_Push -> delete/insert; footprint (none) -> MX_Only:MXOnly-1U
- SW17: value SW_Push -> ~; footprint (none) -> MX_Only:MXOnly-1U
- SW18: value SW_Push -> 1; footprint (none) -> MX_Only:MXOnly-1U
- SW19: value SW_Push -> 2; footprint (none) -> MX_Only:MXOnly-1U
- SW2: value SW_Push -> f1; footprint (none) -> MX_Only:MXOnly-1U
- SW20: value SW_Push -> 3; footprint (none) -> MX_Only:MXOnly-1U
- SW21: value SW_Push -> 4; footprint (none) -> MX_Only:MXOnly-1U
- SW22: value SW_Push -> 5; footprint (none) -> MX_Only:MXOnly-1U
- SW23: value SW_Push -> 6; footprint (none) -> MX_Only:MXOnly-1U
- SW24: value SW_Push -> 7; footprint (none) -> MX_Only:MXOnly-1U
- SW25: value SW_Push -> 8; footprint (none) -> MX_Only:MXOnly-1U
- SW26: value SW_Push -> 9; footprint (none) -> MX_Only:MXOnly-1U
- SW27: value SW_Push -> 0; footprint (none) -> MX_Only:MXOnly-1U
- SW28: value SW_Push -> -; footprint (none) -> MX_Only:MXOnly-1U
- SW29: value SW_Push -> =; footprint (none) -> MX_Only:MXOnly-1U
- SW3: value SW_Push -> f2; footprint (none) -> MX_Only:MXOnly-1U
- SW30: value SW_Push -> backspace; footprint (none) -> MX_Only:MXOnly-2U
- SW31: value SW_Push -> home; footprint (none) -> MX_Only:MXOnly-1U
- SW32: value SW_Push -> tab; footprint (none) -> MX_Only:MXOnly-1.5U
- SW33: value SW_Push -> q; footprint (none) -> MX_Only:MXOnly-1U
- SW34: value SW_Push -> w; footprint (none) -> MX_Only:MXOnly-1U
- SW35: value SW_Push -> e; footprint (none) -> MX_Only:MXOnly-1U
- SW36: value SW_Push -> r; footprint (none) -> MX_Only:MXOnly-1U
- SW37: value SW_Push -> t; footprint (none) -> MX_Only:MXOnly-1U
- SW38: value SW_Push -> y; footprint (none) -> MX_Only:MXOnly-1U
- SW39: value SW_Push -> u; footprint (none) -> MX_Only:MXOnly-1U
- SW4: value SW_Push -> f3; footprint (none) -> MX_Only:MXOnly-1U
- SW40: value SW_Push -> i; footprint (none) -> MX_Only:MXOnly-1U
- SW41: value SW_Push -> o; footprint (none) -> MX_Only:MXOnly-1U
- SW42: value SW_Push -> p; footprint (none) -> MX_Only:MXOnly-1U
- SW43: value SW_Push -> [; footprint (none) -> MX_Only:MXOnly-1U
- SW44: value SW_Push -> ]; footprint (none) -> MX_Only:MXOnly-1U
- SW45: value SW_Push -> \; footprint (none) -> MX_Only:MXOnly-1.5U
- SW46: value SW_Push -> page up; footprint (none) -> MX_Only:MXOnly-1U
- SW47: value SW_Push -> caps lock; footprint (none) -> MX_Only:MXOnly-1.75U
- SW48: value SW_Push -> a; footprint (none) -> MX_Only:MXOnly-1U
- SW49: value SW_Push -> s; footprint (none) -> MX_Only:MXOnly-1U
- SW5: value SW_Push -> f4; footprint (none) -> MX_Only:MXOnly-1U
- SW50: value SW_Push -> d; footprint (none) -> MX_Only:MXOnly-1U
- SW51: value SW_Push -> f; footprint (none) -> MX_Only:MXOnly-1U
- SW52: value SW_Push -> g; footprint (none) -> MX_Only:MXOnly-1U
- SW53: value SW_Push -> h; footprint (none) -> MX_Only:MXOnly-1U
- SW54: value SW_Push -> j; footprint (none) -> MX_Only:MXOnly-1U
- SW55: value SW_Push -> k; footprint (none) -> MX_Only:MXOnly-1U
- SW56: value SW_Push -> l; footprint (none) -> MX_Only:MXOnly-1U
- SW57: value SW_Push -> ;; footprint (none) -> MX_Only:MXOnly-1U
- SW58: value SW_Push -> '; footprint (none) -> MX_Only:MXOnly-1U
- SW59: value SW_Push -> enter; footprint (none) -> MX_Only:MXOnly-2.25U
- SW6: value SW_Push -> f5; footprint (none) -> MX_Only:MXOnly-1U
- SW60: value SW_Push -> page down; footprint (none) -> MX_Only:MXOnly-1U
- SW61: value SW_Push -> shift; footprint (none) -> MX_Only:MXOnly-2.25U
- SW62: value SW_Push -> z; footprint (none) -> MX_Only:MXOnly-1U
- SW63: value SW_Push -> x; footprint (none) -> MX_Only:MXOnly-1U
- SW64: value SW_Push -> c; footprint (none) -> MX_Only:MXOnly-1U
- SW65: value SW_Push -> v; footprint (none) -> MX_Only:MXOnly-1U
- SW66: value SW_Push -> b; footprint (none) -> MX_Only:MXOnly-1U
- SW67: value SW_Push -> n; footprint (none) -> MX_Only:MXOnly-1U
- SW68: value SW_Push -> m; footprint (none) -> MX_Only:MXOnly-1U
- SW69: value SW_Push -> ,; footprint (none) -> MX_Only:MXOnly-1U
- SW7: value SW_Push -> f6; footprint (none) -> MX_Only:MXOnly-1U
- SW70: value SW_Push -> .; footprint (none) -> MX_Only:MXOnly-1U
- SW71: value SW_Push -> /; footprint (none) -> MX_Only:MXOnly-1U
- SW72: value SW_Push -> shift; footprint (none) -> MX_Only:MXOnly-1.75U
- SW73: value SW_Push -> up arrow; footprint (none) -> MX_Only:MXOnly-1U
- SW74: value SW_Push -> end; footprint (none) -> MX_Only:MXOnly-1U
- SW75: value SW_Push -> ctrl; footprint (none) -> MX_Only:MXOnly-1.25U
- SW76: value SW_Push -> win; footprint (none) -> MX_Only:MXOnly-1.25U
- SW77: value SW_Push -> alt; footprint (none) -> MX_Only:MXOnly-1.25U
- SW78: value SW_Push -> space; footprint (none) -> MX_Only:MXOnly-6.25U
- SW79: value SW_Push -> alt; footprint (none) -> MX_Only:MXOnly-1U
- SW8: value SW_Push -> f7; footprint (none) -> MX_Only:MXOnly-1U
- SW80: value SW_Push -> fn; footprint (none) -> MX_Only:MXOnly-1U
- SW81: value SW_Push -> ctrl; footprint (none) -> MX_Only:MXOnly-1U
- SW82: value SW_Push -> left arrow; footprint (none) -> MX_Only:MXOnly-1U
- SW83: value SW_Push -> down arrow; footprint (none) -> MX_Only:MXOnly-1U
- SW84: value SW_Push -> right arrow; footprint (none) -> MX_Only:MXOnly-1U
- SW9: value SW_Push -> f8; footprint (none) -> MX_Only:MXOnly-1U
Connections:
- net col0: now also SW1.2, SW17.2, SW32.2, SW47.2, SW61.2, SW75.2
- net col1: now also SW18.2, SW2.2, SW33.2, SW48.2, SW62.2, SW76.2
- net col10: now also SW11.2, SW27.2, SW42.2, SW57.2, SW71.2, SW79.2
- net col11: now also SW12.2, SW28.2, SW43.2, SW58.2, SW72.2, SW80.2
- net col12: now also SW13.2, SW29.2, SW44.2, SW59.2, SW73.2, SW81.2
- net col13: now also SW14.2, SW30.2, SW45.2, SW82.2
- net col14: now also SW15.2, SW83.2
- net col15: now also SW16.2, SW31.2, SW46.2, SW60.2, SW74.2, SW84.2
- net col2: now also SW19.2, SW3.2, SW34.2, SW49.2, SW63.2, SW77.2
- net col3: now also SW20.2, SW35.2, SW4.2, SW50.2, SW64.2
- net col4: now also SW21.2, SW36.2, SW5.2, SW51.2, SW65.2
- net col5: now also SW22.2, SW37.2, SW52.2, SW6.2, SW66.2
- net col6: now also SW23.2, SW38.2, SW53.2, SW67.2, SW7.2, SW78.2
- net col7: now also SW24.2, SW39.2, SW54.2, SW68.2, SW8.2
- net col8: now also SW25.2, SW40.2, SW55.2, SW69.2, SW9.2
- net col9: now also SW10.2, SW26.2, SW41.2, SW56.2, SW70.2

Commit message: routed columns
Connections:
- net col10: now also SW80.2; no longer SW79.2
- net col11: now also SW81.2; no longer SW80.2
- net col12: no longer SW59.2, SW73.2, SW81.2
- net col13: no longer SW30.2, SW45.2
- net col14: now also SW30.2, SW45.2, SW59.2, SW73.2
- net col9: now also SW79.2
Other:
- moved on the sheet: D30, D45, D59, D73, D79, D80, D81, SW30, SW45, SW59, SW73, SW79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
