File: matrix.kicad_sch (KiCad schematic)
At the start: 168 parts, among them SW1 esc, SW10 f9, SW11 f10, SW12 f11, SW13 f12, SW14 prtsc/nmlk, SW15 pause/scrlk, SW16 delete/insert, SW18 1, SW19 2, SW2 f1, SW20 3, SW21 4, SW22 5, SW23 6, SW24 7, SW25 8, SW26 9, SW27 0, SW28 -, SW29 =, SW3 f2, SW30 backspace, SW31 home, SW32 tab, SW33 q, SW34 w, SW35 e, SW36 r, SW37 t, SW38 y, SW39 u, SW4 f3, SW40 i, SW41 o, SW42 p, SW43 [, SW44 ], SW45 \, SW46 page up, SW47 caps lock, SW48 a, SW49 s, SW5 f4, SW50 d, SW51 f, SW52 g, SW53 h, SW54 j, SW55 k, SW56 l, SW57 ;, SW58 ', SW59 enter, SW6 f5, SW60 page down, SW61 shift, SW62 z, SW63 x, SW64 c, SW65 v, SW66 b, SW67 n, SW68 m, SW69 ,, SW7 f6, SW70 ., SW71 /, SW72 shift, SW73 up arrow, SW74 end, SW75 ctrl, SW76 win, SW77 alt, SW78 space, SW79 alt, SW8 f7, SW80 fn, SW81 ctrl, SW82 left arrow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

Commit message: finished pcb
Connections:
- net col5: now also SW78.2
- net col6: no longer SW78.2
Other:
- moved on the sheet: D78, SW78
Changed lines of the file:
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@@
 	)
 	(junction
+		(at 115.57 116.84)
+		(diameter 0)
+		(color 0 0 0 0)
+	)
+	(junction
 		(at 151.13 85.09)
 		(diameter 0)
@@
 	)
 	(junction
-		(at 118.11 142.24)
+		(at 101.6 142.24)
 		(diameter 0)
 		(color 0 0 0 0)
@@
 	)
 	(junction
-		(at 132.08 116.84)
-		(diameter 0)
-		(color 0 0 0 0)
-	)
-	(junction
 		(at 99.06 41.91)
 		(diameter 0)
@@
 	(wire
 		(pts
-			(xy 132.08 116.84) (xy 132.08 135.89)
+			(xy 115.57 116.84) (xy 115.57 135.89)
 		)
 		(stroke
@@
 	(wire
 		(pts
-			(xy 118.11 140.97) (xy 118.11 142.24)
+			(xy 101.6 140.97) (xy 101.6 142.24)
 		)
 		(stroke
@@
 	(wire
 		(pts
-			(xy 52.07 142.24) (xy 118.11 142.24)
+			(xy 52.07 142.24) (xy 101.6 142.24)
 		)
 		(stroke
@@
 	(wire
 		(pts
-			(xy 118.11 142.24) (xy 167.64 142.24)
-		)
-		(stroke
-			(width 0)
-			(type default)
-		)
-	)
-	(wire
-		(pts
 			(xy 128.27 78.74) (xy 132.08 78.74)
 		)
@@
 	(wire
 		(pts
-			(xy 128.27 135.89) (xy 132.08 135.89)
+			(xy 111.76 135.89) (xy 115.57 135.89)
 		)
 		(stroke
@@
 	(wire
 		(pts
+			(xy 101.6 142.24) (xy 167.64 142.24)
+		)
+		(stroke
+			(width 0)
+			(type default)
+		)
+	)
+	(wire
+		(pts
 			(xy 82.55 97.79) (xy 82.55 116.84)
 		)
@@
 	(symbol
 		(lib_id "Device:D_Small")
-		(at 118.11 138.43 90)
+		(at 101.6 138.43 90)
 		(unit 1)
 		(exclude_from_sim no)
@@
 		(fields_autoplaced yes)
 		(property "Reference" "D78"
-			(at 120.65 137.1599 90)
+			(at 104.14 137.1599 90)
 			(effects
 				(font
@@
 		)
 		(property "Value" "D_Small"
-			(at 120.65 139.6999 90)
+			(at 104.14 139.6999 90)
 			(effects
 				(font
@@
 		)
 		(property "Footprint" "Diode_SMD:D_SOD-123"
-			(at 118.11 138.43 90)
+			(at 101.6 138.43 90)
 			(effects
 				(font
@@
 		)
 		(property "Datasheet" "~"
-			(at 118.11 138.43 90)
+			(at 101.6 138.43 90)
 			(effects
 				(font
@@
 		)
 		(property "Description" "Diode, small symbol"
-			(at 118.11 138.43 0)
+			(at 101.6 138.43 0)
 			(effects
 				(font
@@
 		)
 		(property "Sim.Device" "D"
-			(at 118.11 138.43 0)
+			(at 101.6 138.43 0)
 			(effects
 				(font
@@
 		)
 		(property "Sim.Pins" "1=K 2=A"
-			(at 118.11 138.43 0)
+			(at 101.6 138.43 0)
 			(effects
 				(font
@@
 		)
 		(instances
-			(project ""
+			(project "macropad-from-scratch"
 				(path "/0fae814a-d850-41c2-80ee-052b623b3a63/ae3e0c04-4055-44b5-a7a2-97d160698966"
 					(reference "SW1")
@@
 	(symbol
 		(lib_id "Switch:SW_Push")
-		(at 123.19 135.89 0)
+		(at 106.68 135.89 0)
 		(unit 1)
 		(exclude_from_sim no)
@@
 		(fields_autoplaced yes)
 		(property "Reference" "SW78"
-			(at 123.19 128.27 0)
+			(at 106.68 128.27 0)
 			(effects
 				(font
@@
 		)
 		(property "Value" "space"
-			(at 123.19 130.81 0)
+			(at 106.68 130.81 0)
 			(effects
 				(font
@@
 		)
 		(property "Footprint" "MX_Only:MXOnly-6.25U"
-			(at 123.19 130.81 0)
+			(at 106.68 130.81 0)
 			(effects
 				(font
@@
 		)
 		(property "Datasheet" "~"
-			(at 123.19 130.81 0)
+			(at 106.68 130.81 0)
 			(effects
 				(font
@@
 		)
 		(property "Description" "Push button switch, generic, two pins"
-			(at 123.19 135.89 0)
+			(at 106.68 135.89 0)
 			(effects
 				(font
@@
 		)
 		(instances
-			(project ""
+			(project "macropad-from-scratch"
 				(path "/0fae814a-d850-41c2-80ee-052b623b3a63/ae3e0c04-4055-44b5-a7a2-97d160698966"
 					(reference "D1")
