File: macropad-from-scratch.kicad_pcb (KiCad board)
At the start: 2 copper layers, 189 parts, among them J1 AVR-ISP-6, SW1 esc, SW10 f9, SW11 f10, SW12 f11, SW13 f12, SW14 prtsc/nmlk, SW15 pause/scrlk, SW16 delete/insert, SW18 1, SW19 2, SW2 f1, SW20 3, SW21 4, SW22 5, SW23 6, SW24 7, SW25 8, SW26 9, SW27 0, SW28 -, SW29 =, SW3 f2, SW30 backspace, SW31 home, SW32 tab, SW33 q, SW34 w, SW35 e, SW36 r, SW37 t, SW38 y, SW39 u, SW4 f3, SW40 i, SW41 o, SW42 p, SW43 [, SW44 ], SW45 \, SW46 page up, SW47 caps lock, SW48 a, SW49 s, SW5 f4, SW50 d, SW51 f, SW52 g, SW53 h, SW54 j, SW55 k, SW56 l, SW57 ;, SW58 ', SW59 enter, SW6 f5, SW60 page down, SW61 shift, SW62 z, SW63 x, SW64 c, SW65 v, SW66 b, SW67 n, SW68 m, SW69 ,, SW7 f6, SW70 ., SW71 /, SW72 shift, SW73 up arrow, SW74 end, SW75 ctrl, SW76 win, SW77 alt, SW78 space, SW79 alt, SW8 f7, SW80 fn, SW81 ctrl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

Commit message: routed columns
Parts:
- moved R2 45.6 mm to (252.8, 108.1)
- moved U1 45.3 mm to (249.7, 114.4)
- moved R1 45.2 mm to (248.1, 108.1)
- moved R4 45.0 mm to (254.6, 187.6)
- moved R3 44.6 mm to (251.3, 187.6)
- moved C2 44.2 mm to (273.1, 204.2)
- moved D19 43.2 mm to (148.0, 128.3)
- moved D21 43.2 mm to (186.1, 128.3)
- moved D23 43.2 mm to (224.2, 128.3)
- moved D24 43.2 mm to (243.2, 128.3)
- moved D26 43.2 mm to (281.3, 128.3)
- moved D27 43.2 mm to (300.4, 128.3)
- moved D29 43.2 mm to (338.5, 128.3)
- moved D31 43.2 mm to (395.6, 128.3)
- moved D49 43.2 mm to (162.2, 166.4)
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Connections:
- SW30 pad 2: col13 -> col14
- SW45 pad 2: col13 -> col14
- SW59 pad 2: col12 -> col14
- SW73 pad 2: col12 -> col14
- SW79 pad 2: col10 -> col9
- SW80 pad 2: col11 -> col10
- SW81 pad 2: col12 -> col11
Routing:
- net col11: track 0.00 -> 114.1 mm
- net col2: track 0.00 -> 112.9 mm
- net col1: track 0.00 -> 112.9 mm
- net col14: track 0.00 -> 111.0 mm
- net col10: track 0.00 -> 107.9 mm
- net col9: track 0.00 -> 107.1 mm
- net col0: track 0.00 -> 105.2 mm
- net col13: track 0.00 -> 96.7 mm
- net col15: track 0.00 -> 95.2 mm
- net col5: track 0.00 -> 88.6 mm
- net col7: track 0.00 -> 86.1 mm
- net col8: track 0.00 -> 86.1 mm
- net col6: track 0.00 -> 86.1 mm
- net col3: track 0.00 -> 86.1 mm
- net col4: track 0.00 -> 86.1 mm
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Other:
- board outline added: 304.8 x 119.9 mm

Commit message: routed the matrix
Parts:
- moved U1 8.87 mm to (248.1, 105.7)
- moved R1 7.82 mm to (243.5, 101.8)
- moved C2 6.90 mm to (268.1, 199.4), turned to 0 degrees
- moved C1 6.09 mm to (268.1, 202.6), turned to 0 degrees
- moved Y1 3.68 mm to (263.8, 200.8), turned to 90 degrees
- moved C3 1.14 mm to (262.6, 195.4)
- moved USB1 0.44 mm to (248.3, 90.8)
- moved D16 0.32 mm to (395.9, 108.9)
Routing:
- net row0: track 0.00 -> 271.5 mm
- net row1: track 0.00 -> 271.1 mm
- net row2: track 0.00 -> 266.3 mm
- net row3: track 0.00 -> 263.8 mm
- net row4: track 0.00 -> 259.1 mm
- net row5: track 0.00 -> 217.0 mm
- net /D+: track 0.00 -> 101.3 mm
- net /D-: track 0.00 -> 100.0 mm
- net GND: track 0.00 -> 25.1 mm
- net Net-(D16-A): track 0.00 -> 14.1 mm
- net /XTAL1: track 0.00 -> 13.3 mm
- net Net-(D82-A): track 0.00 -> 13.2 mm
- net Net-(D79-A): track 0.00 -> 13.1 mm
- net Net-(D5-A): track 0.00 -> 12.8 mm
- net Net-(D59-A): track 0.00 -> 12.8 mm
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