File: macropad-from-scratch.kicad_pcb (KiCad board)
At the start: 2 copper layers, 304.8 x 119.9 mm, 189 parts, among them J1 AVR-ISP-6, SW1 esc, SW10 f9, SW11 f10, SW12 f11, SW13 f12, SW14 prtsc/nmlk, SW15 pause/scrlk, SW16 delete/insert, SW18 1, SW19 2, SW2 f1, SW20 3, SW21 4, SW22 5, SW23 6, SW24 7, SW25 8, SW26 9, SW27 0, SW28 -, SW29 =, SW3 f2, SW30 backspace, SW31 home, SW32 tab, SW33 q, SW34 w, SW35 e, SW36 r, SW37 t, SW38 y, SW39 u, SW4 f3, SW40 i, SW41 o, SW42 p, SW43 [, SW44 ], SW45 \, SW46 page up, SW47 caps lock, SW48 a, SW49 s, SW5 f4, SW50 d, SW51 f, SW52 g, SW53 h, SW54 j, SW55 k, SW56 l, SW57 ;, SW58 ', SW59 enter, SW6 f5, SW60 page down, SW61 shift, SW62 z, SW63 x, SW64 c, SW65 v, SW66 b, SW67 n, SW68 m, SW69 ,, SW7 f6, SW70 ., SW71 /, SW72 shift, SW73 up arrow, SW74 end, SW75 ctrl, SW76 win, SW77 alt, SW78 space, SW79 alt, SW8 f7, SW80 fn, SW81 ctrl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

Commit message: finished pcb
Parts:
- added FB1: 60@100MHz, Inductor_SMD:L_0805_2012Metric_Pad1.05x1.20mm_HandSolder, B.Cu at (259.8, 97.0)
- added REF**: MountingHole_2.2mm_M2, MountingHole:MountingHole_2.2mm_M2, F.Cu at (118.9, 200.4)
- added REF**: MountingHole_2.2mm_M2, MountingHole:MountingHole_2.2mm_M2, F.Cu at (380.8, 104.9)
- added REF**: MountingHole_2.2mm_M2, MountingHole:MountingHole_2.2mm_M2, F.Cu at (114.1, 100.2)
- added REF**: MountingHole_2.2mm_M2, MountingHole:MountingHole_2.2mm_M2, F.Cu at (380.8, 200.4)
- moved J1 77.5 mm to (284.0, 191.5), turned to 90 degrees
- moved R1 9.05 mm to (250.7, 107.3), turned to 0 degrees
- moved R2 8.89 mm to (245.9, 102.6), turned to 180 degrees
- moved R7 8.24 mm to (275.9, 200.4)
- moved U1 4.81 mm to (248.3, 110.5)
- moved SW85 2.71 mm to (283.2, 200.2), turned to 180 degrees
- moved F1 1.92 mm to (245.1, 114.5)
- moved C4 1.11 mm to (258.6, 206.5)
- moved R8 1.11 mm to (245.0, 206.5)
- moved C5 1.11 mm to (257.2, 189.9), turned to 90 degrees
- moved R4 0.79 mm to (253.8, 187.6)
- moved R3 0.22 mm to (251.5, 187.5)
- turned C8 to 180 degrees
Connections:
- R3 pad 2: Net-(U2-D-) -> /D-
- R4 pad 2: Net-(U2-D+) -> /D+
- SW78 pad 2: col6 -> col5
- U2 pad 1: row0 -> row4
- U2 pad 3: Net-(U2-D-) -> /D-
- U2 pad 36: col5 -> row5
- U2 pad 37: row5 -> col5
- U2 pad 38: row4 -> row0
- U2 pad 39: row3 -> row1
- U2 pad 4: Net-(U2-D+) -> /D+
- U2 pad 41: row1 -> row3
- USB1 pad 13: GND -> Earth
Routing:
- net GND: track 25.1 -> 299.1 mm, vias 0 -> 100
- net row0: track 271.5 -> 523.9 mm, vias 0 -> 2
- net row1: track 271.1 -> 498.4 mm, vias 0 -> 2
- net row2: track 266.3 -> 474.3 mm, vias 0 -> 2
- net +5V: track 6.18 -> 208.2 mm, vias 0 -> 9
- net row3: track 263.8 -> 449.7 mm, vias 0 -> 2
- net col15: track 95.2 -> 253.3 mm, vias 0 -> 1
- net col0: track 105.2 -> 262.0 mm, vias 0 -> 1
- net col12: track 42.0 -> 197.9 mm, vias 0 -> 1
- net row4: track 259.1 -> 413.0 mm, vias 0 -> 4
- net col14: track 111.0 -> 248.4 mm, vias 0 -> 1
- net col1: track 112.9 -> 242.9 mm, vias 0 -> 1
- net col13: track 96.7 -> 213.1 mm, vias 0 -> 1
- net col2: track 112.9 -> 215.2 mm, vias 0 -> 1
- net row5: track 217.0 -> 308.6 mm
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- added copper zone on B.Cu, net Earth
- added copper zone on F.Cu, net Earth
- added copper zone on B.Cu, net GND
- added copper zone on F.Cu, net GND
