File: macropad-from-scratch.kicad_sch (KiCad schematic)
At the start: 21 parts, among them J1 AVR-ISP-6, SW85 SW_Push, U1 PRTR5V0U2X, U2 ATmega32U4-A, Y1 Crystal_GND24_Small

Commit message: finished pcb
Parts:
- added FB1: 60@100MHz, Inductor_SMD:L_0805_2012Metric_Pad1.05x1.20mm_HandSolder, symbol Device:FerriteBead_Small
Connections:
- net D+: now also R4.2, U2.4 (D+); no longer R4.1, U1.2 (IO1), USB1.6 (DP1), USB1.8 (DP2)
- net D-: now also R3.2, U2.3 (D-); no longer R3.1, U1.3 (IO2), USB1.5 (DN2), USB1.7 (DN1)
- net GND: now also FB1.2; no longer USB1.13 (SHIELD)
- net col5: now also U2.37 (PF6); no longer U2.36 (PF7)
- net row0: now also U2.38 (PF5); no longer U2.1 (PE6)
- net row1: now also U2.39 (PF4); no longer U2.41 (PF0)
- net row3: now also U2.41 (PF0); no longer U2.39 (PF4)
- net row4: now also U2.1 (PE6); no longer U2.38 (PF5)
- net row5: now also U2.36 (PF7); no longer U2.37 (PF6)
- new net: R4.1, U1.2 (IO1), USB1.6 (DP1), USB1.8 (DP2)
- new net: R3.1, U1.3 (IO2), USB1.5 (DN2), USB1.7 (DN1)
- new net Earth: FB1.1, USB1.13 (SHIELD)
Other:
- moved on the sheet: R3, R4
